File: schematics/usb host hub/usb host hub/usb host hub.kicad_sch (KiCad schematic)
At the start: 56 parts, among them J1 292303-1, J2 292303-1, J4 Conn_01x04_Male, J5 Conn_01x04_Male, J6 292303-1, U1 RP2040, U2 FE1.1s, U3 W25Q128JVS, U4 AZ1117EH-3.3TRG1, U5 USBLC6-2SC6, U6 USBLC6-2SC6, U7 USBLC6-2SC6, Y1 12MHz, Y2 12MHz

Commit message: Rv32: Rev 2 USB Host schematics. Ordered from JLCPCB.
Parts:
- removed C18: 27pF, Capacitor_SMD:C_0805_2012Metric, symbol Device:C_Small
- added R14, R15: 33k, Resistor_SMD:R_0805_2012Metric, symbol Device:R_Small
- added TP_1V1, TP_DRV1, TP_LED1, TP_LED2: TestPoint_Small, TestPoint:TestPoint_Pad_D1.5mm, symbol Connector:TestPoint_Small
- C17: value 27pF -> 100nF; footprint Capacitor_SMD:C_0805_2012Metric -> Capacitor_SMD:C_0402_1005Metric; LCSC (none) -> C307331
- R11: value 33 -> 47
- R12: value 1k -> 33k
Connections:
- net +1V1: now also TP_1V1.1
- net GND: now also R12.2, R14.2, R15.2; no longer U2.27 (TESTJ/EESDA)
- net VD18: now also C17.1
- net at J1.SH1 (SHIELD), J1.SH2 (SHIELD): now also R14.1
- net at J6.SH1 (SHIELD), J6.SH2 (SHIELD): now also R12.1
- net at U2.2 (XOUT): now also Y2.1; no longer R12.2
- net at J2.SH1 (SHIELD), J2.SH2 (SHIELD): now also R15.1
- net DRV: now reaches U2.22 (DRV)
- net DRV: now also TP_DRV1.1
- net LED1: now reaches U2.23 (LED1/EESCL)
- net LED1: now also TP_LED1.1
- net LED2: now reaches U2.24 (LED2)
- net LED2: now also TP_LED2.1
- no-connect marks 38 -> 33
Other:
- note added: "Rev 2"
- moved on the sheet: C19, C20
